File: AR_20_JW_Rev2/AR_20_JW_Rev2.sch (KiCad schematic (older format))
At the start: 14 parts

Commit message: Completed PCB model and manufacturing files Generated Gerber files Changed hole placement for mounting Completed traces for PCB Chose footprints for all components
Parts:
- C1, C2: renamed from C?; value 22pF -> 20pF; footprint (none) -> Capacitor_THT:C_Rect_L7.2mm_W3.0mm_P5.00mm_FKS2_FKP2_MKS2_MKP2
- J1: renamed from J?; footprint (none) -> LED_SMD:LED_1206_3216Metric
- R1, R3, R5: renamed from R?; value 1M -> 5k; footprint (none) -> Resistor_SMD:R_1206_3216Metric
- R2: renamed from R?; value 1M -> 85 Ohm; footprint (none) -> Resistor_SMD:R_1206_3216Metric
- R4: renamed from R?; value R -> 5k; footprint (none) -> Resistor_SMD:R_1206_3216Metric
- U2: renamed from U?; footprint (none) -> Connector_PinHeader_2.54mm:PinHeader_2x03_P2.54mm_Vertical; symbol AR_20_JW:ICSP -> AR_20_JW_Rev2-rescue:ICSP-AR_20_JW
- U3: renamed from U?; footprint (none) -> Connector_PinHeader_2.54mm:PinHeader_1x07_P2.54mm_Vertical; symbol AR_20_JW:MCP2515_CAN -> AR_20_JW_Rev2-rescue:MCP2515_CAN-AR_20_JW
- U4: renamed from U?; footprint (none) -> Connector_PinHeader_2.54mm:PinHeader_1x06_P2.54mm_Vertical; symbol AR_20_JW:INPUT -> AR_20_JW_Rev2-rescue:INPUT-AR_20_JW
- U5: renamed from U?; footprint (none) -> Connector_PinHeader_2.54mm:PinHeader_1x06_P2.54mm_Vertical; symbol AR_20_JW:SWITCH -> AR_20_JW_Rev2-rescue:SWITCH-AR_20_JW
- Y1: renamed from Y?; value Crystal -> 16 MHz Crystal; footprint (none) -> Crystal:Crystal_SMD_HC49-SD_HandSoldering
- gave numbers to parts that had none: 1
Connections:
- wire segments 68 -> 69
Other:
- moved on the sheet: C1, C2, J1, R1, R2, R3, R4, R5, U1, Y1

Commit message: Initial Commit
Created 3 new headders for the different inputs for the board
Created AER branch
Parts:
- removed R3, R4, R5: 5k, Resistor_SMD:R_1206_3216Metric, symbol Device:R
- removed U4: INPUT, Connector_PinHeader_2.54mm:PinHeader_1x06_P2.54mm_Vertical, symbol AR_20_JW_Rev2-rescue:INPUT-AR_20_JW
- removed U5: SWITCH, Connector_PinHeader_2.54mm:PinHeader_1x06_P2.54mm_Vertical, symbol AR_20_JW_Rev2-rescue:SWITCH-AR_20_JW
- added U? (x4): RIDE, symbol AR_20_JW_Rev2-rescue:RIDE
- added U?: STR, symbol AR_20_JW_Rev2-rescue:RIDE
- added U? (x4): SPD, symbol AR_20_JW_Rev2-rescue:SPD_1
- U1: symbol MCU_Microchip_ATmega:ATmega328P-PU -> AR_20_JW_Rev2-rescue:ATmega328P-PU-MCU_Microchip_ATmega
Connections:
- net AUX_1: no longer names the net of U1.13 (PD7)
- net AUX_2: no longer names the net of U1.14 (PB0)
- net FDB_SIG: no longer names the net of U1.23 (PC0)
- net SIG_CNT: no longer names the net of U1.11 (PD5)
- net SIG_EXT: no longer names the net of U1.12 (PD6)
- net SIG_RUN: no longer names the net of U1.6 (PD4)
- net TX_1: no longer names the net of U1.3 (PD1)
